Commit message: j1 j2 ok

File: urdf/nero_description.urdf (robot description, URDF)
Before this commit: robot nero, 9 links, 8 joints
Joints:
- joint joint1: limit lower=-2.70526 upper=2.70526 effort=100 velocity=5 -> lower=-2.7401669256 upper=2.7401669256 effort=100 velocity=3.1415926536
- joint joint2: limit lower=-1.74 upper=1.74 effort=100 velocity=5 -> lower=-0.2617993878 upper=3.3161255788 effort=100 velocity=3.1415926536
- joint joint3: limit lower=-2.75 upper=2.75 effort=100 velocity=5 -> lower=-2.7925268032 upper=2.7925268032 effort=100 velocity=3.1415926536
- joint joint4: limit lower=-1.01 upper=2.14 effort=100 velocity=5 -> lower=-1.0471975512 upper=2.1816615650 effort=100 velocity=3.9269908170
- joint joint5: limit lower=-2.75 upper=2.75 effort=100 velocity=5 -> lower=-2.7925268032 upper=2.7925268032 effort=100 velocity=3.9269908170
- joint joint6: limit lower=-0.73 upper=0.95 effort=100 velocity=5 -> lower=-0.7504915784 upper=1.0122909662 effort=100 velocity=3.9269908170
- joint joint7: limit lower=-1.5707963 upper=1.5707963 effort=100 velocity=5 -> lower=-1.5707963268 upper=1.5707963268 effort=100 velocity=3.9269908170
