Commit message: 人体朝向与动作深度

File: urdf/nero_description.urdf (robot description, URDF)
Before this commit: robot nero, 9 links, 8 joints
Links:
- link base_link: geometry collision mesh filename=package://armbycontroller/agx_arm_urdf/nero/meshes/base_lin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; visual mesh filename=package://armbycontroller/agx_arm_urdf/nero/meshes/dae/base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
- link link1: geometry collision mesh filename=package://armbycontroller/agx_arm_urdf/nero/meshes/link1.stl; visual mesh filename=package://armbycontroller/agx_arm_urdf/nero/meshes/dae/link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
- link link2: geometry collision mesh filename=package://armbycontroller/agx_arm_urdf/nero/meshes/link2.stl; visual mesh filename=package://armbycontroller/agx_arm_urdf/nero/meshes/dae/link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
- link link3: geometry collision mesh filename=package://armbycontroller/agx_arm_urdf/nero/meshes/link3.stl; visual mesh filename=package://armbycontroller/agx_arm_urdf/nero/meshes/dae/link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
- link link4: geometry collision mesh filename=package://armbycontroller/agx_arm_urdf/nero/meshes/link4.stl; visual mesh filename=package://armbycontroller/agx_arm_urdf/nero/meshes/dae/link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
- link link5: geometry collision mesh filename=package://armbycontroller/agx_arm_urdf/nero/meshes/link5.stl; visual mesh filename=package://armbycontroller/agx_arm_urdf/nero/meshes/dae/link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
- link link6: geometry collision mesh filename=package://armbycontroller/agx_arm_urdf/nero/meshes/link6.stl; visual mesh filename=package://armbycontroller/agx_arm_urdf/nero/meshes/dae/link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
- link link7: geometry collision mesh filename=package://armbycontroller/agx_arm_urdf/nero/meshes/link7.stl; visual mesh filename=package://armbycontroller/agx_arm_urdf/nero/meshes/dae/link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

File: urdf/nero_with_left_revo2_description.xacro (robot description, xacro)
@@ -4,6 +4,6 @@
      For more information, please see http://wiki.ros.org/sw_urdf_exporter -->
 <robot xmlns:xacro="http://www.ros.org/wiki/xacro" name="nero">
-<xacro:include filename="$(find agx_arm_description)/agx_arm_urdf/revo2/urdf/revo2_left_hand.urdf"/>
-<xacro:include filename="$(find agx_arm_description)/agx_arm_urdf/nero/urdf/nero_with_revo2_flange_description.xacro"/>
+<xacro:include filename="$(find armbycontroller)/agx_arm_urdf/revo2/urdf/revo2_left_hand.urdf"/>
+<xacro:include filename="$(find armbycontroller)/agx_arm_urdf/nero/urdf/nero_with_revo2_flange_description.xacro"/>
     <joint name="hand_base_joint" type="fixed">
         <origin xyz="0.0 0.0 0.012" rpy="0 0 3.1415926"/>

File: urdf/nero_with_right_revo2_description.xacro (robot description, xacro)
@@ -4,6 +4,6 @@
      For more information, please see http://wiki.ros.org/sw_urdf_exporter -->
 <robot xmlns:xacro="http://www.ros.org/wiki/xacro" name="nero">
-<xacro:include filename="$(find agx_arm_description)/agx_arm_urdf/revo2/urdf/revo2_right_hand.urdf"/>
-<xacro:include filename="$(find agx_arm_description)/agx_arm_urdf/nero/urdf/nero_with_revo2_flange_description.xacro"/>
+<xacro:include filename="$(find armbycontroller)/agx_arm_urdf/revo2/urdf/revo2_right_hand.urdf"/>
+<xacro:include filename="$(find armbycontroller)/agx_arm_urdf/nero/urdf/nero_with_revo2_flange_description.xacro"/>
     <joint name="hand_base_joint" type="fixed">
         <origin xyz="0.0 0.0 0.012" rpy="0 0 3.1415926"/>
